Commit message: convert livox_ros2_driver submodule to normal folder

File: src/rm_robot_description/urdf/sentry.urdf.xacro (robot description, xacro)
@@ -18,7 +18,5 @@
     <origin xyz = "0 0 -0.722" rpy = "0 0 0"/>
   </joint>
-</robot>
-  <!-- <link name="gimbal_imu" /> -->
-  <!-- <link name="gimbal_link" />
+   <link name="gimbal_link" />
   <joint name="gimbal_joint" type="floating">
     <parent link="livox_frame" />
@@ -37,3 +35,5 @@
     <parent link="camera_link" />
     <child link="camera_optical_frame" />
-  </joint> -->
+  </joint>
+</robot>
+  <!-- <link name="gimbal_imu" /> -->
